File: HeatBoard.kicad_pcb (KiCad board)
At the start: 2 copper layers, 19 parts, among them J81 J8HeaderTurned, J82 J8Header, Q1 BC337, Q2 BC337

Commit message: First Final
Parts:
- moved R2 24.1 mm to (209.6, 142.2), turned to 90 degrees
- moved R1 2.84 mm to (215.9, 142.2)
Connections:
- R2 pad 1: Net-(Bu1-Pad1) -> Net-(Co1-Pad1)
Routing:
- net Net-(Bu1-Pad1): track 505.1 -> 496.2 mm
- net Net-(Co1-Pad2): track 97.5 -> 104.6 mm
- net Net-(C1-Pad1): track 299.7 -> 297.7 mm
- net Net-(Co3-Pad2): track 63.2 -> 64.9 mm
- net Net-(Co1-Pad1): track 134.9 -> 136.5 mm
- net Net-(Co2-Pad2): track 72.9 -> 73.7 mm
- net Net-(J81-Pad34): track 59.6 -> 58.8 mm

Commit message: Raspi Connections move, GND Pin free now
Parts:
- moved J81 16.7 mm to (168.9, 121.9)
- moved J82 7.41 mm to (205.7, 113.0)
- moved Co3 2.54 mm to (227.3, 152.4)
- moved Co1 2.54 mm to (215.9, 152.4)
- moved Co2 2.54 mm to (238.8, 152.4)
- moved R1 2.54 mm to (218.4, 142.2)
- moved R2 2.54 mm to (212.1, 142.2)
- moved R4 2.54 mm to (221.0, 127.0)
Connections:
- J81 pad 36: Net-(Co2-Pad2) -> Net-(J81-Pad36)
- J81 pad 38: Net-(Co3-Pad2) -> Net-(Co2-Pad2)
- J81 pad 40: Net-(J81-Pad40) -> Net-(Co3-Pad2)
- J82 pad 36: Net-(Co2-Pad2) -> Net-(J81-Pad36)
- J82 pad 38: Net-(Co3-Pad2) -> Net-(Co2-Pad2)
- J82 pad 40: Net-(J81-Pad40) -> Net-(Co3-Pad2)
- R3 pad 1: Net-(J81-Pad34) -> Net-(J81-Pad32)
- R4 pad 1: Net-(J81-Pad32) -> Net-(J81-Pad36)
- RL1 pad 7: Net-(RL1-Pad7) -> Net-(Co4-Pad2)
- RL1 pad 8: Net-(RL1-Pad8) -> Net-(F2-Pad1)
Routing:
- net Net-(Bu1-Pad1): track 496.2 -> 422.7 mm
- net Net-(J81-Pad36): track 0.00 -> 55.7 mm
- net Net-(Co1-Pad2): track 104.6 -> 138.9 mm
- net Net-(J81-Pad32): track 35.0 -> 68.3 mm
- net Net-(Co1-Pad1): track 136.5 -> 168.3 mm
- net Net-(J81-Pad28): track 20.1 -> 44.1 mm
- net Net-(J81-Pad8): track 20.1 -> 44.1 mm
- net Net-(J81-Pad16): track 20.1 -> 44.1 mm
- net Net-(J81-Pad4): track 20.1 -> 44.1 mm
- net Net-(J81-Pad30): track 20.1 -> 44.1 mm
- net Net-(J81-Pad24): track 20.1 -> 44.1 mm
- net Net-(J81-Pad22): track 20.1 -> 44.1 mm
- net Net-(J81-Pad20): track 20.1 -> 44.1 mm
- net Net-(J81-Pad39): track 14.0 -> 38.0 mm
- net Net-(J81-Pad33): track 14.0 -> 38.0 mm
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